File: micr0x/Hardware/micr0x.brd (EAGLE design)
At the start: 160 x 24 mm, 29 parts, among them IC1 SN74HC174DR, IC2 LM358D, IC3 CD4066BPWR, Q1 2SC1623-L6-TP, Q2 2SC1623-L6-TP

Commit message: added interface section
Parts:
- added C10, C11, C3, C4, C5, C6, C7, C8, C9: 0.1uF, SamacSys_Parts:CAPC1608X90N
- added C2: 1uF, rcl:E2-5
- added D1, D2: 1N4148, diode:DO35-7
- added IC10, IC12, IC13, IC14, IC9: 74HC595D, 74xx-eu:SO16
- added IC11, IC7, IC8: 74HC165D, 74xx-eu:SO16
- added IC4: ATMEGA162-16AU, SamacSys_Parts:QFP80P1200X1200X120-44N
- added IC5: SN74HC126D, SamacSys_Parts:SOIC127P600X175-14N
- added IC6: AT25P, atmel:DIL08
- added LED1, LED10, LED11, LED12, LED13, LED14, LED15, LED16, LED2, LED3, LED4, LED5, LED6, LED7, LED8, LED9: (no value), led:LED3MM
- added Q3: (no value), murata-resonators:CSTLS_X
- added R24: 1M, rcl:R0603
- added R25, R26, R27, R28, R29, R30, R31, R32, R41, R42, R43, R44, R45, R46, R47, R48, R57, R58, R59, R60, R61, R62, R63, R64: 10k, rcl:R0603
- added R33, R34, R35, R36, R37, R38, R39, R40, R49, R50, R51, R52, R53, R54, R55, R56, R65, R66, R67, R68, R69, R70, R71, R72, R73, R74, R75, R76, R77, R78, R79, R80, R81, R82, R83, R84, R85, R86, R87, R88: 10, rcl:R0603
- added S1, S10, S11, S12, S13, S14, S15, S16, S17, S18, S19, S2, S20, S21, S22, S23, S24, S3, S4, S5, S6, S7, S8, S9: ITSFV1, its-switch:ITSFV1
- moved R21 25.4 mm to (48.3, 3.81)
- moved R22 25.4 mm to (53.3, 3.81)
- moved R23 25.4 mm to (58.4, 3.81)
Connections:
- new net BUF_1A: C2.+, D1.A, D2.C, IC5.2, R24.1
- new net BUF_1Y: D2.A, IC4.4, IC5.3
- new net BUF_3A: IC5.9, IC7.9
- new net GND_1: IC4.28
- new net GND_2: IC4.39
- new net LED_LATCH: IC10.12, IC12.12, IC13.12, IC14.12, IC4.30, IC9.12
- new net N$100: IC13.7, R80.1
- new net N$101: R65.2, S17.L2
- new net N$102: R66.2, S18.L2
- new net N$103: R67.2, S19.L2
- new net N$104: R68.2, S20.L2
- new net N$105: R69.2, S21.L2
- new net N$106: R70.2, S22.L2
- new net N$107: R71.2, S23.L2
- new net N$108: R72.2, S24.L2
- new net N$109: IC12.7, R72.1
- new net N$110: IC12.6, R71.1
- new net N$111: IC12.5, R70.1
- new net N$112: IC12.4, R69.1
- new net N$113: IC12.3, R68.1
- new net N$114: IC12.2, R67.1
- new net N$115: IC12.1, R66.1
- new net N$116: IC12.15, R65.1
- new net N$117: IC13.6, R79.1
- new net N$118: IC13.5, R78.1
- new net N$119: IC13.4, R77.1
- new net N$120: IC13.3, R76.1
- new net N$121: IC13.2, R75.1
- new net N$122: IC13.1, R74.1
- new net N$123: IC13.15, R73.1
- new net N$124: LED1.A, R73.2
- new net N$125: LED2.A, R74.2
- new net N$126: LED3.A, R75.2
- new net N$127: LED4.A, R76.2
- new net N$128: LED5.A, R77.2
- new net N$129: LED6.A, R78.2
- new net N$130: LED7.A, R79.2
- new net N$131: LED8.A, R80.2
- new net N$132: IC14.7, R88.1
- new net N$133: IC14.6, R87.1
- new net N$134: IC14.5, R86.1
- new net N$135: IC14.4, R85.1
- new net N$136: IC14.3, R84.1
- new net N$137: IC14.2, R83.1
- new net N$138: IC14.1, R82.1
- new net N$139: IC14.15, R81.1
- new net N$140: LED9.A, R81.2
- new net N$141: LED10.A, R82.2
- new net N$142: LED11.A, R83.2
- new net N$143: LED12.A, R84.2
- new net N$144: LED13.A, R85.2
- new net N$145: LED14.A, R86.2
- new net N$146: LED15.A, R87.2
- new net N$147: LED16.A, R88.2
- new net N$16: IC4.14, Q3.1
- new net N$17: IC4.15, Q3.3
- new net N$18: IC7.6, S1.2
- new net N$19: IC7.5, S2.2
- new net N$20: IC7.4, S3.2
- new net N$21: IC7.3, S4.2
- new net N$22: IC7.11, S8.2
- new net N$23: IC7.12, S7.2
- new net N$24: IC7.13, S6.2
- new net N$25: IC7.14, S5.2
- new net N$26: R25.2, S1.1
- new net N$27: R26.2, S2.1
- new net N$28: R27.2, S3.1
- new net N$29: R28.2, S4.1
- new net N$30: R29.2, S5.1
- new net N$31: R30.2, S6.1
- new net N$32: R31.2, S7.1
- new net N$33: R32.2, S8.1
- new net N$34: R33.2, S1.L2
- new net N$35: R34.2, S2.L2
- new net N$36: R35.2, S3.L2
- new net N$37: R36.2, S4.L2
- new net N$38: R37.2, S5.L2
- new net N$39: R38.2, S6.L2
- new net N$40: R39.2, S7.L2
- new net N$41: R40.2, S8.L2
- new net N$42: IC10.7, R40.1
- new net N$43: IC10.6, R39.1
- new net N$44: IC10.5, R38.1
- new net N$45: IC10.4, R37.1
- new net N$46: IC10.3, R36.1
- new net N$47: IC10.2, R35.1
- new net N$48: IC10.1, R34.1
- new net N$49: IC10.15, R33.1
- new net N$50: IC8.6, S9.2
- new net N$51: IC8.5, S10.2
- new net N$52: IC8.4, S11.2
- new net N$53: IC8.3, S12.2
- new net N$54: IC8.11, S16.2
- new net N$55: IC8.12, S15.2
- new net N$56: IC8.13, S14.2
- new net N$57: IC8.14, S13.2
- new net N$58: R41.2, S9.1
- new net N$59: R42.2, S10.1
- new net N$60: R43.2, S11.1
- new net N$61: R44.2, S12.1
- new net N$62: R45.2, S13.1
- new net N$63: R46.2, S14.1
- new net N$64: R47.2, S15.1
- new net N$65: R48.2, S16.1
- new net N$66: IC7.10, IC8.9
- new net N$67: IC11.9, IC8.10
- new net N$68: R49.2, S9.L2
- new net N$69: R50.2, S10.L2
- new net N$70: R51.2, S11.L2
- new net N$71: R52.2, S12.L2
- new net N$72: R53.2, S13.L2
- new net N$73: R54.2, S14.L2
- new net N$74: R55.2, S15.L2
- new net N$75: R56.2, S16.L2
- new net N$76: IC9.7, R56.1
- new net N$77: IC9.6, R55.1
- new net N$78: IC9.5, R54.1
- new net N$79: IC9.4, R53.1
- new net N$80: IC9.3, R52.1
- new net N$81: IC9.2, R51.1
- new net N$82: IC9.1, R50.1
- new net N$83: IC9.15, R49.1
- new net N$84: IC11.6, S17.2
- new net N$85: IC11.5, S18.2
- new net N$86: IC11.4, S19.2
- new net N$87: IC11.3, S20.2
- new net N$88: IC11.11, S24.2
- new net N$89: IC11.12, S23.2
- new net N$90: IC11.13, S22.2
- new net N$91: IC11.14, S21.2
- new net N$92: R57.2, S17.1
- new net N$93: R58.2, S18.1
- new net N$94: R59.2, S19.1
- new net N$95: R60.2, S20.1
- new net N$96: R61.2, S21.1
- new net N$97: R62.2, S22.1
- new net N$98: R63.2, S23.1
- new net N$99: R64.2, S24.1
- new net SPI_CLK: IC10.11, IC11.2, IC12.11, IC13.11, IC14.11, IC4.3, IC6.6, IC7.2, IC8.2, IC9.11
- new net SPI_IN: IC6.5
- new net SPI_OUT: IC5.8, IC6.2
- new net SWITCH_LATCH: IC11.1, IC5.10, IC6.1, IC7.1, IC8.1
- new net VCC_1: IC4.17
- new net VCC_2: IC4.38
- net GND: now also C10.1, C11.1, C2.-, C3.1, C4.1, C5.1, C6.1, C7.1, C8.1, C9.1, IC10.13, IC10.8, IC11.10, IC11.15, IC11.8, IC12.13, IC12.8, IC13.13, IC13.8, IC14.13, IC14.8, IC4.16, IC5.7, IC6.4, IC7.15, IC7.8, IC8.15, IC8.8, IC9.13, IC9.8, LED1.K, LED10.K, LED11.K, LED12.K, LED13.K, LED14.K, LED15.K, LED16.K, LED2.K, LED3.K, LED4.K, LED5.K, LED6.K, LED7.K, LED8.K, LED9.K, Q3.2, R25.1, R26.1, R27.1, R28.1, R29.1, R30.1, R31.1, R32.1, R41.1, R42.1, R43.1, R44.1, R45.1, R46.1, R47.1, R48.1, R57.1, R58.1, R59.1, R60.1, R61.1, R62.1, R63.1, R64.1, S1.L1, S10.L1, S11.L1, S12.L1, S13.L1, S14.L1, S15.L1, S16.L1, S17.L1, S18.L1, S19.L1, S2.L1, S20.L1, S21.L1, S22.L1, S23.L1, S24.L1, S3.L1, S4.L1, S5.L1, S6.L1, S7.L1, S8.L1, S9.L1
- net VCC: now also C10.2, C11.2, C3.2, C4.2, C5.2, C6.2, C7.2, C8.2, C9.2, D1.C, IC10.10, IC10.16, IC11.16, IC12.10, IC12.16, IC13.10, IC13.16, IC14.10, IC14.16, IC4.6, IC5.1, IC5.14, IC6.3, IC6.7, IC6.8, IC7.16, IC8.16, IC9.10, IC9.16, R24.2, S1.3, S10.3, S11.3, S12.3, S13.3, S14.3, S15.3, S16.3, S17.3, S18.3, S19.3, S2.3, S20.3, S21.3, S22.3, S23.3, S24.3, S3.3, S4.3, S5.3, S6.3, S7.3, S8.3, S9.3
Other:
- board size 160 x 24 mm -> 240 x 24 mm

Commit message: add components
Parts:
- added C12: 10uF, rcl:E2-5
- added C13: 0.1uF, SamacSys_Parts:CAPC1608X90N
- added D3: 1N4148, diode:DO35-7
- added R89: 22k, rcl:R0603
- added R90, R91, R92, R93: 10k, rcl:R0603
- added R94: 1k, rcl:R0603
- added R95, R96, R97: 100k, rcl:R0603
- added T1, T3: 2SC536F, transistor:TO92
- added T2: 2SA733P, transistor:TO92
- moved C4 17.3 mm to (64.8, -34.3)
- moved C6 17.3 mm to (11.4, -34.3)
- moved IC10 17.3 mm to (17.8, -30.5)
- moved R33 17.3 mm to (25.4, -35.6)
- moved R34 17.3 mm to (30.5, -35.6)
- moved R35 17.3 mm to (35.6, -35.6)
- moved R36 17.3 mm to (40.6, -35.6)
- moved R37 17.3 mm to (45.7, -35.6)
- moved R38 17.3 mm to (50.8, -35.6)
- moved R39 17.3 mm to (55.9, -35.6)
- moved R40 17.3 mm to (61.0, -35.6)
Connections:
- net N$4 renamed CV_OUT
- removed net GND_1: IC4.28
- new net ACCENT: IC4.19, R95.1
- new net ACCENT_OUT: R97.1, T3.3
- new net GATE: IC4.27, R89.1
- new net GATE_OUT: R94.2
- new net N$148: C12.-, R91.2, R92.1, T2.2
- new net N$149: R91.1, T1.3
- new net N$150: R89.2, R90.2, T1.2
- new net N$151: D3.A, R93.2, T2.3
- new net N$152: D3.C, R94.1
- new net N$153: R95.2, R96.2, T3.2
- net GND: now also C13.1, IC4.28, R90.1, R93.1, R96.1, T1.1, T3.1
- net NOTE0: now also IC4.20
- net NOTE1: now also IC4.21
- net NOTE2: now also IC4.22
- net NOTE3: now also IC4.23
- net NOTE4: now also IC4.24
- net NOTE5: now also IC4.25
- net SLIDE: now also IC4.18
- net SPI_IN: now also IC4.1
- net SPI_OUT: now also IC4.2
- net VCC: now also C12.+, C13.2, R92.2, R97.2, T2.1

Commit message: add change
Connections:
- removed net N$13: IC1.9
- new net NOTE_LATCH: IC1.9, IC4.26
Changed lines of the file:
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@@
 <wire x1="10.345" y1="9.525" x2="226.742921875" y2="15.06880625" width="0" layer="19" extent="1-16"/>
-</signal>
-<signal name="N$13">
-<contactref element="IC1" pad="9"/>
 </signal>
 <signal name="N$14">
@@
 <wire x1="69.85" y1="-47.41" x2="69.85" y2="-52.49" width="0" layer="19" extent="1-1"/>
 </signal>
+<signal name="NOTE_LATCH">
+<contactref element="IC4" pad="26"/>
+<contactref element="IC1" pad="9"/>
+<wire x1="10.345" y1="6.985" x2="226.1772375" y2="9.76550625" width="0" layer="19" extent="1-16"/>
+</signal>
 </signals>
