File: micr0x/Hardware/micr0x.sch (EAGLE design)
At the start: 29 parts, among them IC1 SN74HC174DR, IC2 LM358D, IC3 CD4066BPWR, Q1 2SC1623-L6-TP, Q2 2SC1623-L6-TP

Commit message: added interface section
Parts:
- added C10, C11, C3, C4, C5, C6, C7, C8, C9: 0.1uF, SamacSys_Parts:GCJ188R71H104KA12D
- added C2: 1uF, rcl:CPOL-EUE2-5
- added D1, D2: 1N4148, diode:1N4148DO35-7
- added IC10, IC12, IC13, IC14, IC9: 74HC595D, 74xx-eu:74HC595D
- added IC11, IC7, IC8: 74HC165D, 74xx-eu:74HC165D
- added IC4: ATMEGA162-16AU, SamacSys_Parts:ATMEGA162-16AU
- added IC5: SN74HC126D, SamacSys_Parts:SN74HC126D
- added IC6: AT25P, atmel:AT25P
- added LED1, LED10, LED11, LED12, LED13, LED14, LED15, LED16, LED2, LED3, LED4, LED5, LED6, LED7, LED8, LED9: (no value), led:LED3MM
- added Q3: (no value), murata-resonators:CSTLS_X
- added R24: 1M, rcl:R-EU_R0603
- added R25, R26, R27, R28, R29, R30, R31, R32, R41, R42, R43, R44, R45, R46, R47, R48, R57, R58, R59, R60, R61, R62, R63, R64: 10k, rcl:R-EU_R0603
- added R33, R34, R35, R36, R37, R38, R39, R40, R49, R50, R51, R52, R53, R54, R55, R56, R65, R66, R67, R68, R69, R70, R71, R72, R73, R74, R75, R76, R77, R78, R79, R80, R81, R82, R83, R84, R85, R86, R87, R88: 10, rcl:R-EU_R0603
- added S1, S10, S11, S12, S13, S14, S15, S16, S17, S18, S19, S2, S20, S21, S22, S23, S24, S3, S4, S5, S6, S7, S8, S9: ITSFV1, its-switch:ITSFV1
Connections:
- new net BUF_1A: C2.+, D1.A, D2.C, IC5.1A, R24.1
- new net BUF_1Y: D2.A, IC4.!RESET, IC5.1Y
- new net BUF_3A: IC5.3A, IC7A.QH
- new net LED_LATCH: IC10A.RCK, IC12A.RCK, IC13A.RCK, IC14A.RCK, IC4.PA7_[AD7/PCINT7], IC9A.RCK
- new net N$100: IC13A.QH, R80.1
- new net N$101: R65.2, S17LED.L2
- new net N$102: R66.2, S18LED.L2
- new net N$103: R67.2, S19LED.L2
- new net N$104: R68.2, S20LED.L2
- new net N$105: R69.2, S21LED.L2
- new net N$106: R70.2, S22LED.L2
- new net N$107: R71.2, S23LED.L2
- new net N$108: R72.2, S24LED.L2
- new net N$109: IC12A.QH, R72.1
- new net N$110: IC12A.QG, R71.1
- new net N$111: IC12A.QF, R70.1
- new net N$112: IC12A.QE, R69.1
- new net N$113: IC12A.QD, R68.1
- new net N$114: IC12A.QC, R67.1
- new net N$115: IC12A.QB, R66.1
- new net N$116: IC12A.QA, R65.1
- new net N$117: IC13A.QG, R79.1
- new net N$118: IC13A.QF, R78.1
- new net N$119: IC13A.QE, R77.1
- new net N$120: IC13A.QD, R76.1
- new net N$121: IC13A.QC, R75.1
- new net N$122: IC13A.QB, R74.1
- new net N$123: IC13A.QA, R73.1
- new net N$124: LED1.A, R73.2
- new net N$125: LED2.A, R74.2
- new net N$126: LED3.A, R75.2
- new net N$127: LED4.A, R76.2
- new net N$128: LED5.A, R77.2
- new net N$129: LED6.A, R78.2
- new net N$130: LED7.A, R79.2
- new net N$131: LED8.A, R80.2
- new net N$132: IC14A.QH, R88.1
- new net N$133: IC14A.QG, R87.1
- new net N$134: IC14A.QF, R86.1
- new net N$135: IC14A.QE, R85.1
- new net N$136: IC14A.QD, R84.1
- new net N$137: IC14A.QC, R83.1
- new net N$138: IC14A.QB, R82.1
- new net N$139: IC14A.QA, R81.1
- new net N$140: LED9.A, R81.2
- new net N$141: LED10.A, R82.2
- new net N$142: LED11.A, R83.2
- new net N$143: LED12.A, R84.2
- new net N$144: LED13.A, R85.2
- new net N$145: LED14.A, R86.2
- new net N$146: LED15.A, R87.2
- new net N$147: LED16.A, R88.2
- new net N$16: IC4.XTAL2, Q3.1
- new net N$17: IC4.XTAL1, Q3.3
- new net N$18: IC7A.H, S1SW.2
- new net N$19: IC7A.G, S2SW.2
- new net N$20: IC7A.F, S3SW.2
- new net N$21: IC7A.E, S4SW.2
- new net N$22: IC7A.A, S8SW.2
- new net N$23: IC7A.B, S7SW.2
- new net N$24: IC7A.C, S6SW.2
- new net N$25: IC7A.D, S5SW.2
- new net N$26: R25.2, S1SW.1
- new net N$27: R26.2, S2SW.1
- new net N$28: R27.2, S3SW.1
- new net N$29: R28.2, S4SW.1
- new net N$30: R29.2, S5SW.1
- new net N$31: R30.2, S6SW.1
- new net N$32: R31.2, S7SW.1
- new net N$33: R32.2, S8SW.1
- new net N$34: R33.2, S1LED.L2
- new net N$35: R34.2, S2LED.L2
- new net N$36: R35.2, S3LED.L2
- new net N$37: R36.2, S4LED.L2
- new net N$38: R37.2, S5LED.L2
- new net N$39: R38.2, S6LED.L2
- new net N$40: R39.2, S7LED.L2
- new net N$41: R40.2, S8LED.L2
- new net N$42: IC10A.QH, R40.1
- new net N$43: IC10A.QG, R39.1
- new net N$44: IC10A.QF, R38.1
- new net N$45: IC10A.QE, R37.1
- new net N$46: IC10A.QD, R36.1
- new net N$47: IC10A.QC, R35.1
- new net N$48: IC10A.QB, R34.1
- new net N$49: IC10A.QA, R33.1
- new net N$50: IC8A.H, S9SW.2
- new net N$51: IC8A.G, S10SW.2
- new net N$52: IC8A.F, S11SW.2
- new net N$53: IC8A.E, S12SW.2
- new net N$54: IC8A.A, S16SW.2
- new net N$55: IC8A.B, S15SW.2
- new net N$56: IC8A.C, S14SW.2
- new net N$57: IC8A.D, S13SW.2
- new net N$58: R41.2, S9SW.1
- new net N$59: R42.2, S10SW.1
- new net N$60: R43.2, S11SW.1
- new net N$61: R44.2, S12SW.1
- new net N$62: R45.2, S13SW.1
- new net N$63: R46.2, S14SW.1
- new net N$64: R47.2, S15SW.1
- new net N$65: R48.2, S16SW.1
- new net N$66: IC7A.SER, IC8A.QH
- new net N$67: IC11A.QH, IC8A.SER
- new net N$68: R49.2, S9LED.L2
- new net N$69: R50.2, S10LED.L2
- new net N$70: R51.2, S11LED.L2
- new net N$71: R52.2, S12LED.L2
- new net N$72: R53.2, S13LED.L2
- new net N$73: R54.2, S14LED.L2
- new net N$74: R55.2, S15LED.L2
- new net N$75: R56.2, S16LED.L2
- new net N$76: IC9A.QH, R56.1
- new net N$77: IC9A.QG, R55.1
- new net N$78: IC9A.QF, R54.1
- new net N$79: IC9A.QE, R53.1
- new net N$80: IC9A.QD, R52.1
- new net N$81: IC9A.QC, R51.1
- new net N$82: IC9A.QB, R50.1
- new net N$83: IC9A.QA, R49.1
- new net N$84: IC11A.H, S17SW.2
- new net N$85: IC11A.G, S18SW.2
- new net N$86: IC11A.F, S19SW.2
- new net N$87: IC11A.E, S20SW.2
- new net N$88: IC11A.A, S24SW.2
- new net N$89: IC11A.B, S23SW.2
- new net N$90: IC11A.C, S22SW.2
- new net N$91: IC11A.D, S21SW.2
- new net N$92: R57.2, S17SW.1
- new net N$93: R58.2, S18SW.1
- new net N$94: R59.2, S19SW.1
- new net N$95: R60.2, S20SW.1
- new net N$96: R61.2, S21SW.1
- new net N$97: R62.2, S22SW.1
- new net N$98: R63.2, S23SW.1
- new net N$99: R64.2, S24SW.1
- new net SPI_CLK: IC10A.SCK, IC11A.CLK, IC12A.SCK, IC13A.SCK, IC14A.SCK, IC4.[SCK]_PB7, IC6.SCK, IC7A.CLK, IC8A.CLK, IC9A.SCK
- new net SPI_IN: IC6.SI
- new net SPI_OUT: IC5.3Y, IC6.SO
- new net SWITCH_LATCH: IC11A.SH/!LD, IC5.3OE, IC6.CS/, IC7A.SH/!LD, IC8A.SH/!LD
- net GND: now also C10.1, C11.1, C2.-, C3.1, C4.1, C5.1, C6.1, C7.1, C8.1, C9.1, IC10A.G, IC11A.INH, IC11A.SER, IC12A.G, IC13A.G, IC14A.G, IC5.GND, IC6.GND, IC7A.INH, IC8A.INH, IC9A.G, LED1.C, LED10.C, LED11.C, LED12.C, LED13.C, LED14.C, LED15.C, LED16.C, LED2.C, LED3.C, LED4.C, LED5.C, LED6.C, LED7.C, LED8.C, LED9.C, Q3.VSS, R25.1, R26.1, R27.1, R28.1, R29.1, R30.1, R31.1, R32.1, R41.1, R42.1, R43.1, R44.1, R45.1, R46.1, R47.1, R48.1, R57.1, R58.1, R59.1, R60.1, R61.1, R62.1, R63.1, R64.1, S10LED.L1, S11LED.L1, S12LED.L1, S13LED.L1, S14LED.L1, S15LED.L1, S16LED.L1, S17LED.L1, S18LED.L1, S19LED.L1, S1LED.L1, S20LED.L1, S21LED.L1, S22LED.L1, S23LED.L1, S24LED.L1, S2LED.L1, S3LED.L1, S4LED.L1, S5LED.L1, S6LED.L1, S7LED.L1, S8LED.L1, S9LED.L1
- net VCC: now also C10.2, C11.2, C3.2, C4.2, C5.2, C6.2, C7.2, C8.2, C9.2, D1.C, IC10A.SCL, IC12A.SCL, IC13A.SCL, IC14A.SCL, IC5.1OE, IC5.VCC, IC6.HOLD/, IC6.VCC, IC6.WP/, IC9A.SCL, R24.2, S10SW.3, S11SW.3, S12SW.3, S13SW.3, S14SW.3, S15SW.3, S16SW.3, S17SW.3, S18SW.3, S19SW.3, S1SW.3, S20SW.3, S21SW.3, S22SW.3, S23SW.3, S24SW.3, S2SW.3, S3SW.3, S4SW.3, S5SW.3, S6SW.3, S7SW.3, S8SW.3, S9SW.3

Commit message: add components
Parts:
- added C12: 10uF, rcl:CPOL-EUE2-5
- added C13: 0.1uF, SamacSys_Parts:GCJ188R71H104KA12D
- added D3: 1N4148, diode:1N4148DO35-7
- added R89: 22k, rcl:R-EU_R0603
- added R90, R91, R92, R93: 10k, rcl:R-EU_R0603
- added R94: 1k, rcl:R-EU_R0603
- added R95, R96, R97: 100k, rcl:R-EU_R0603
- added T1, T3: 2SC536F, transistor:-NPN-TO92
- added T2: 2SA733P, transistor:-PNP-TO92
Connections:
- net N$4 renamed CV_OUT
- new net ACCENT: IC4.[A9/PCINT9]_PC1, R95.1
- new net ACCENT_OUT: R97.1, T3.C
- new net GATE: IC4.PE1_[ALE], R89.1
- new net GATE_OUT: R94.2
- new net N$148: C12.-, R91.2, R92.1, T2.B
- new net N$149: R91.1, T1.C
- new net N$150: R89.2, R90.2, T1.B
- new net N$151: D3.A, R93.2, T2.C
- new net N$152: D3.C, R94.1
- new net N$153: R95.2, R96.2, T3.B
- net GND: now also C13.1, IC4.GND, IC4.GND_1, R90.1, R93.1, R96.1, T1.E, T3.E
- net NOTE0: now also IC4.[A10/PCINT10]_PC2
- net NOTE1: now also IC4.[A11/PCINT11]_PC3
- net NOTE2: now also IC4.[TCK/A12/PCINT12]_PC4
- net NOTE3: now also IC4.PC5_[A13/TMS/PCINT13]
- net NOTE4: now also IC4.PC6_[A14/TDO/PCINT14]
- net NOTE5: now also IC4.PC7_[A15/TDI/PCINT15]
- net SLIDE: now also IC4.[A8/PCINT8]_PC0
- net SPI_IN: now also IC4.[MOSI]_PB5
- net SPI_OUT: now also IC4.[MISO]_PB6
- net VCC: now also C12.+, C13.2, IC4.VCC, R92.2, R97.2, T2.E
Other:
- moved on the sheet: C1, C10, C11, C2, C3, C4, C5, C6, C7, C8, C9, D1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

Commit message: add change
Connections:
- removed net N$13: IC1.CLK
- new net NOTE_LATCH: IC1.CLK, IC4.PE2_[OC1B]
Changed lines of the file:
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@@
 <setting verticaltext="up"/>
 </settings>
-<grid distance="0.05" unitdist="inch" unit="inch" style="lines" multiple="1" display="yes" altdistance="0.01" altunitdist="inch" altunit="mm"/>
+<grid distance="0.05" unitdist="inch" unit="inch" style="lines" multiple="1" display="no" altdistance="0.01" altunitdist="inch" altunit="inch"/>
 <layers>
 <layer number="1" name="Top" color="4" fill="1" visible="no" active="no"/>
@@
 </segment>
 </net>
-<net name="N$13" class="0">
-<segment>
-<pinref part="IC1" gate="G$1" pin="CLK"/>
-<wire x1="97.79" y1="283.21" x2="100.33" y2="283.21" width="0.1524" layer="91"/>
-</segment>
-</net>
 <net name="N$14" class="0">
 <segment>
@@
 </segment>
 </net>
+<net name="NOTE_LATCH" class="0">
+<segment>
+<pinref part="IC4" gate="G$1" pin="PE2_[OC1B]"/>
+<wire x1="132.08" y1="149.86" x2="147.32" y2="149.86" width="0.1524" layer="91"/>
+<label x="139.7" y="149.86" size="1.778" layer="95"/>
+</segment>
+<segment>
+<pinref part="IC1" gate="G$1" pin="CLK"/>
+<wire x1="97.79" y1="283.21" x2="110.49" y2="283.21" width="0.1524" layer="91"/>
+<label x="100.33" y="283.21" size="1.778" layer="95"/>
+</segment>
+</net>
